Commit message: 采用宇树b1的机器人描述方式，改写a1和f1的模型

File: legged_examples/legged_unitree/legged_unitree_description/urdf/a1/const.xacro (robot description, xacro)
@@ -18,5 +18,5 @@
     <xacro:property name="calf_height" value="0.016"/>
     <xacro:property name="calf_x_offset" value="0.0"/>
-    <xacro:property name="foot_radius" value="0.02"/>
+    <xacro:property name="foot_radius" value="0.03"/>
     <!-- kinematic value -->
     <xacro:property name="thigh_offset" value="0.0838"/>
@@ -28,17 +28,27 @@
     <xacro:property name="trunk_offset_z" value="0.01675"/>
     <xacro:property name="hip_offset" value="0.065"/>
+    <!-- offset of link and rotor locations (left front) -->
+    <xacro:property name="hip_rotor_offset_x" value="0.1"/>
+    <xacro:property name="hip_rotor_offset_y" value="0.05"/>
+    <xacro:property name="hip_rotor_offset_z" value="0.0"/>
+    <xacro:property name="thigh_rotor_offset_x" value="0.0"/>
+    <xacro:property name="thigh_rotor_offset_y" value="0.0"/>
+    <xacro:property name="thigh_rotor_offset_z" value="0.0"/>
+    <xacro:property name="calf_rotor_offset_x" value="0.0"/>
+    <xacro:property name="calf_rotor_offset_y" value="-0.04"/>
+    <xacro:property name="calf_rotor_offset_z" value="0.0"/>
     <!-- joint limits -->
     <xacro:property name="damping" value="0"/>
     <xacro:property name="friction" value="0"/>
-    <xacro:property name="hip_max" value="${46*pi/180.0}"/>
-    <xacro:property name="hip_min" value="${-46*pi/180.0}"/>
+    <xacro:property name="hip_position_max" value="${46*pi/180.0}"/>
+    <xacro:property name="hip_position_min" value="${-46*pi/180.0}"/>
     <xacro:property name="hip_velocity_max" value="21"/>
     <xacro:property name="hip_torque_max" value="33.5"/>
-    <xacro:property name="thigh_max" value="${240*pi/180.0}"/>
-    <xacro:property name="thigh_min" value="${-60*pi/180.0}"/>
+    <xacro:property name="thigh_position_max" value="${240*pi/180.0}"/>
+    <xacro:property name="thigh_position_min" value="${-60*pi/180.0}"/>
     <xacro:property name="thigh_velocity_max" value="21"/>
     <xacro:property name="thigh_torque_max" value="33.5"/>
-    <xacro:property name="calf_max" value="${-52.5*pi/180.0}"/>
-    <xacro:property name="calf_min" value="${-154.5*pi/180.0}"/>
+    <xacro:property name="calf_position_max" value="${-52.5*pi/180.0}"/>
+    <xacro:property name="calf_position_min" value="${-154.5*pi/180.0}"/>
     <xacro:property name="calf_velocity_max" value="21"/>
     <xacro:property name="calf_torque_max" value="33.5"/>
@@ -66,4 +76,14 @@
     <xacro:property name="hip_iyz" value="-0.000000545"/>
     <xacro:property name="hip_izz" value="0.000487919"/>
+    <xacro:property name="hip_rotor_mass" value="0.001"/><!-- 质心相对于hip转子的位置-->
+    <xacro:property name="hip_rotor_com_x" value="0.0"/>
+    <xacro:property name="hip_rotor_com_y" value="0.0"/>
+    <xacro:property name="hip_rotor_com_z" value="0.0"/>
+    <xacro:property name="hip_rotor_ixx" value="0.000103801"/>
+    <xacro:property name="hip_rotor_ixy" value="0.0"/>
+    <xacro:property name="hip_rotor_ixz" value="0.0"/>
+    <xacro:property name="hip_rotor_iyy" value="0.000054638"/>
+    <xacro:property name="hip_rotor_iyz" value="0.0"/>
+    <xacro:property name="hip_rotor_izz" value="0.000054638"/>
     <!-- thigh -->
     <xacro:property name="thigh_mass" value="0.888"/>
@@ -77,4 +97,14 @@
     <xacro:property name="thigh_iyz" value="-0.000028174"/>
     <xacro:property name="thigh_izz" value="0.001110200"/>
+    <xacro:property name="thigh_rotor_mass" value="0.001"/>
+    <xacro:property name="thigh_rotor_com_x" value="0.0"/>
+    <xacro:property name="thigh_rotor_com_y" value="0.0"/>
+    <xacro:property name="thigh_rotor_com_z" value="0.0"/>
+    <xacro:property name="thigh_rotor_ixx" value="0.000103801"/>
+    <xacro:property name="thigh_rotor_ixy" value="0.0"/>
+    <xacro:property name="thigh_rotor_ixz" value="0.0"/>
+    <xacro:property name="thigh_rotor_iyy" value="0.000054638"/>
+    <xacro:property name="thigh_rotor_iyz" value="0.0"/>
+    <xacro:property name="thigh_rotor_izz" value="0.000054638"/>
     <!-- calf -->
     <xacro:property name="calf_mass" value="0.151"/>
@@ -88,4 +118,14 @@
     <xacro:property name="calf_iyz" value="0.0"/>
     <xacro:property name="calf_izz" value="0.000031158"/>
+    <xacro:property name="calf_rotor_mass" value="0.001"/>
+    <xacro:property name="calf_rotor_com_x" value="0.0"/>
+    <xacro:property name="calf_rotor_com_y" value="0.0"/>
+    <xacro:property name="calf_rotor_com_z" value="0.0"/>
+    <xacro:property name="calf_rotor_ixx" value="0.000103801"/>
+    <xacro:property name="calf_rotor_ixy" value="0.0"/>
+    <xacro:property name="calf_rotor_ixz" value="0.0"/>
+    <xacro:property name="calf_rotor_iyy" value="0.000054638"/>
+    <xacro:property name="calf_rotor_iyz" value="0.0"/>
+    <xacro:property name="calf_rotor_izz" value="0.000054638"/>
     <!-- foot -->
     <xacro:property name="foot_mass" value="0.06"/>

File: legged_examples/legged_unitree/legged_unitree_description/urdf/common/leg.xacro (robot description, xacro)
@@ -2,7 +2,18 @@
 <robot xmlns:xacro="http://www.ros.org/wiki/xacro">
     <xacro:include filename="$(find legged_unitree_description)/urdf/common/transmission.xacro"/>
-    <xacro:macro name="leg" params="prefix mirror mirror_dae front_hind front_hind_dae *origin">
+    <xacro:macro name="leg" params="prefix mirror mirror_dae front_hind front_hind_dae">
         <joint name="${prefix}_HAA" type="revolute">
-            <xacro:insert_block name="origin"/>
+            <xacro:if value="${(mirror_dae == False) and (front_hind_dae == True)}">
+                <origin rpy="0 0 0" xyz="${leg_offset_x} ${-leg_offset_y} 0"/>
+            </xacro:if>
+            <xacro:if value="${(mirror_dae == True) and (front_hind_dae == True)}">
+                <origin rpy="0 0 0" xyz="${leg_offset_x} ${leg_offset_y} 0"/>
+            </xacro:if>
+            <xacro:if value="${(mirror_dae == False) and (front_hind_dae == False)}">
+                <origin rpy="0 0 0" xyz="${-leg_offset_x} ${-leg_offset_y} 0"/>
+            </xacro:if>
+            <xacro:if value="${(mirror_dae == True) and (front_hind_dae == False)}">
+                <origin rpy="0 0 0" xyz="${-leg_offset_x} ${leg_offset_y} 0"/>
+            </xacro:if>
             <parent link="base"/>
             <child link="${prefix}_hip"/>
@@ -10,11 +21,25 @@
             <dynamics damping="${damping}" friction="${friction}"/>
             <xacro:if value="${(mirror_dae == True)}">
-                <limit effort="${hip_torque_max}" velocity="${hip_velocity_max}" lower="${hip_min}"
-                       upper="${hip_max}"/>
+                <limit effort="${hip_torque_max}" velocity="${hip_velocity_max}" lower="${hip_position_min}" upper="${hip_position_max}"/>
             </xacro:if>
             <xacro:if value="${(mirror_dae == False)}">
-                <limit effort="${hip_torque_max}" velocity="${hip_velocity_max}" lower="${-hip_max}"
-                       upper="${-hip_min}"/>
-            </xacro:if>
+                <limit effort="${hip_torque_max}" velocity="${hip_velocity_max}" lower="${-hip_position_max}" upper="${-hip_position_min}"/>
+            </xacro:if>
+        </joint>
+        <joint name="${prefix}_HAA_rotor" type="fixed">
+            <xacro:if value="${(mirror_dae == False) and (front_hind_dae == True)}">
+                <origin rpy="0 0 0" xyz="${hip_rotor_offset_x} ${-hip_rotor_offset_y} 0"/>
+            </xacro:if>
+            <xacro:if value="${(mirror_dae == True) and (front_hind_dae == True)}">
+                <origin rpy="0 0 0" xyz="${hip_rotor_offset_x} ${hip_rotor_offset_y} 0"/>
+            </xacro:if>
+            <xacro:if value="${(mirror_dae == False) and (front_hind_dae == False)}">
+                <origin rpy="0 0 0" xyz="${-hip_rotor_offset_x} ${-hip_rotor_offset_y} 0"/>
+            </xacro:if>
+            <xacro:if value="${(mirror_dae == True) and (front_hind_dae == False)}">
+                <origin rpy="0 0 0" xyz="${-hip_rotor_offset_x} ${hip_rotor_offset_y} 0"/>
+            </xacro:if>
+            <parent link="trunk"/>
+            <child link="${prefix}_hip_rotor"/>
         </joint>
         <link name="${prefix}_hip">
@@ -51,4 +76,27 @@
                         iyy="${hip_iyy}" iyz="${hip_iyz*mirror}"
                         izz="${hip_izz}"/>
+            </inertial>
+        </link>
+        <link name="${prefix}_hip_rotor">
+            <visual>
+                <origin rpy="0 ${pi/2.0} 0" xyz="0 0 0"/>
+                <geometry>
+                    <cylinder length="0.015" radius="0.03"/>
+                </geometry>
+                <material name="green"/>
+            </visual>
+            <!-- <collision>
+                <origin rpy="0 ${pi/2.0} 0" xyz="0 0 0"/>
+                <geometry>
+                    <cylinder length="0.02" radius="0.05"/>
+                </geometry>
+            </collision> -->
+            <inertial>
+                <origin rpy="0 0 0" xyz="${hip_rotor_com_x} ${hip_rotor_com_y} ${hip_rotor_com_z}"/>
+                <mass value="${hip_rotor_mass}"/>
+                <inertia
+                        ixx="${hip_rotor_ixx}" ixy="${hip_rotor_ixy}" ixz="${hip_rotor_ixz}"
+                        iyy="${hip_rotor_iyy}" iyz="${hip_rotor_iyz}"
+                        izz="${hip_rotor_izz}"/>
             </inertial>
         </link>
@@ -59,6 +107,10 @@
             <axis xyz="0 1 0"/>
             <dynamics damping="${damping}" friction="${friction}"/>
-            <limit effort="${thigh_torque_max}" velocity="${thigh_velocity_max}" lower="${thigh_min}"
-                   upper="${thigh_max}"/>
+            <limit effort="${thigh_torque_max}" velocity="${thigh_velocity_max}" lower="${thigh_position_min}" upper="${thigh_position_max}"/>
+        </joint>
+        <joint name="${prefix}_HFE_rotor" type="fixed">
+            <origin rpy="0 0 0" xyz="${thigh_rotor_offset_x} ${thigh_rotor_offset_y*mirror} 0"/>
+            <parent link="${prefix}_hip"/>
+            <child link="${prefix}_thigh_rotor"/>
         </joint>
         <link name="${prefix}_thigh">
@@ -67,10 +119,8 @@
                 <geometry>
                     <xacro:if value="${mirror_dae == True}">
-                        <mesh filename="package://legged_unitree_description/meshes/$(arg robot_type)/thigh.dae"
-                              scale="1 1 1"/>
+                        <mesh filename="package://legged_unitree_description/meshes/$(arg robot_type)/thigh.dae" scale="1 1 1"/>
                     </xacro:if>
                     <xacro:if value="${mirror_dae == False}">
-                        <mesh filename="package://legged_unitree_description/meshes/$(arg robot_type)/thigh_mirror.dae"
-                              scale="1 1 1"/>
+                        <mesh filename="package://legged_unitree_description/meshes/$(arg robot_type)/thigh_mirror.dae" scale="1 1 1"/>
                     </xacro:if>
                 </geometry>
@@ -78,5 +128,5 @@
             </visual>
             <collision>
-                <origin rpy="0 ${pi/2.0+0.1} 0" xyz="${thigh_x_offset} 0 ${-thigh_length/2.0}"/>
+                <origin rpy="0 ${pi/2.0} 0" xyz="${thigh_x_offset} 0 ${-thigh_length/2.0}"/>
                 <geometry>
                     <box size="${thigh_length} ${thigh_width} ${thigh_height}"/>
@@ -96,4 +146,27 @@
                         iyy="${thigh_iyy}" iyz="${thigh_iyz*mirror}"
                         izz="${thigh_izz}"/>
+            </inertial>
+        </link>
+        <link name="${prefix}_thigh_rotor">
+            <visual>
+                <origin rpy="${pi/2.0} 0 0" xyz="0 0 0"/>
+                <geometry>
+                    <cylinder length="0.015" radius="0.03"/>
+                </geometry>
+                <material name="green"/>
+            </visual>
+            <!-- <collision>
+                <origin rpy="${pi/2.0} 0 0" xyz="0 0 0"/>
+                <geometry>
+                    <cylinder length="0.02" radius="0.05"/>
+                </geometry>
+            </collision> -->
+            <inertial>
+                <origin rpy="0 0 0" xyz="${thigh_rotor_com_x} ${thigh_rotor_com_y} ${thigh_rotor_com_z}"/>
+                <mass value="${thigh_rotor_mass}"/>
+                <inertia
+                        ixx="${thigh_rotor_ixx}" ixy="${thigh_rotor_ixy}" ixz="${thigh_rotor_ixz}"
+                        iyy="${thigh_rotor_iyy}" iyz="${thigh_rotor_iyz}"
+                        izz="${thigh_rotor_izz}"/>
             </inertial>
         </link>
@@ -104,5 +177,10 @@
             <axis xyz="0 1 0"/>
             <dynamics damping="${damping}" friction="${friction}"/>
-            <limit effort="${calf_torque_max}" velocity="${calf_velocity_max}" lower="${calf_min}" upper="${calf_max}"/>
+            <limit effort="${calf_torque_max}" velocity="${calf_velocity_max}" lower="${calf_position_min}" upper="${calf_position_max}"/>
+        </joint>
+        <joint name="${prefix}_KFE_rotor" type="fixed">
+            <origin rpy="0 0 0" xyz="${calf_rotor_offset_x} ${calf_rotor_offset_y*mirror} 0"/>
+            <parent link="${prefix}_thigh"/>
+            <child link="${prefix}_calf_rotor"/>
         </joint>
         <link name="${prefix}_calf">
@@ -110,6 +188,5 @@
                 <origin rpy="0 0 0" xyz="0 0 0"/>
                 <geometry>
-                    <mesh filename="package://legged_unitree_description/meshes/$(arg robot_type)/calf.dae"
-                          scale="1 1 1"/>
+                    <mesh filename="package://legged_unitree_description/meshes/$(arg robot_type)/calf.dae" scale="1 1 1"/>
                 </geometry>
                 <material name="orange"/>
@@ -128,4 +205,27 @@
                         iyy="${calf_iyy}" iyz="${calf_iyz}"
                         izz="${calf_izz}"/>
+            </inertial>
+        </link>
+        <link name="${prefix}_calf_rotor">
+            <visual>
+                <origin rpy="${pi/2.0} 0 0" xyz="0 0 0"/>
+                <geometry>
+                    <cylinder length="0.015" radius="0.03"/>
+                </geometry>
+                <material name="green"/>
+            </visual>
+            <!-- <collision>
+                <origin rpy="${pi/2.0} 0 0" xyz="0 0 0"/>
+                <geometry>
+                    <cylinder length="0.02" radius="0.05"/>
+                </geometry>
+            </collision> -->
+            <inertial>
+                <origin rpy="0 0 0" xyz="${calf_rotor_com_x} ${calf_rotor_com_y} ${calf_rotor_com_z}"/>
+                <mass value="${calf_rotor_mass}"/>
+                <inertia
+                        ixx="${calf_rotor_ixx}" ixy="${calf_rotor_ixy}" ixz="${calf_rotor_ixz}"
+                        iyy="${calf_rotor_iyy}" iyz="${calf_rotor_iyz}"
+                        izz="${calf_rotor_izz}"/>
             </inertial>
         </link>
@@ -141,5 +241,5 @@
                     <sphere radius="${foot_radius-0.01}"/>
                 </geometry>
-                <material name="orange"/>
+                <material name="green"/>
             </visual>
             <collision>

File: legged_examples/legged_unitree/legged_unitree_description/urdf/f1/const.xacro (robot description, xacro)
@@ -5,11 +5,11 @@
     <!-- simplified collision value -->
     <xacro:property name="trunk_width" value="0.32"/>
-    <xacro:property name="trunk_length" value="0.698"/>
+    <xacro:property name="trunk_length" value="0.512"/>
     <xacro:property name="trunk_height" value="0.155"/>
     <xacro:property name="hip_radius" value="0.064"/>
     <xacro:property name="hip_length" value="0.056"/><!-- -->
     <xacro:property name="thigh_shoulder_radius" value="0.064"/>
-    <xacro:property name="thigh_shoulder_length" value="0.134"/>
-    <xacro:property name="thigh_shoulder_y_offset" value="0.1201"/>
+    <xacro:property name="thigh_shoulder_length" value="0.047"/>
+    <xacro:property name="thigh_shoulder_y_offset" value="0.0"/>
     <xacro:property name="thigh_width" value="0.047"/>
     <xacro:property name="thigh_height" value="0.07"/>
@@ -28,17 +28,27 @@
     <xacro:property name="trunk_offset_z" value="0.01675"/>
     <xacro:property name="hip_offset" value="0.1201"/>    <!-- thigh_offset_y-->
+    <!-- offset of link and rotor locations (left front) -->
+    <xacro:property name="hip_rotor_offset_x" value="0.1962"/>
+    <xacro:property name="hip_rotor_offset_y" value="0.094"/>
+    <xacro:property name="hip_rotor_offset_z" value="0.0"/>
+    <xacro:property name="thigh_rotor_offset_x" value="0.0"/>
+    <xacro:property name="thigh_rotor_offset_y" value="-0.03917"/>
+    <xacro:property name="thigh_rotor_offset_z" value="0.0"/>
+    <xacro:property name="calf_rotor_offset_x" value="0.0"/>
+    <xacro:property name="calf_rotor_offset_y" value="-0.08583"/>
+    <xacro:property name="calf_rotor_offset_z" value="0.0"/>
     <!-- joint limits -->
     <xacro:property name="damping" value="0"/>
     <xacro:property name="friction" value="0"/>
-    <xacro:property name="hip_max" value="0.75"/>
-    <xacro:property name="hip_min" value="-0.75"/>
+    <xacro:property name="hip_position_max" value="0.75"/>
+    <xacro:property name="hip_position_min" value="-0.75"/>
     <xacro:property name="hip_velocity_max" value="19.69"/>
     <xacro:property name="hip_torque_max" value="91.0035"/>
-    <xacro:property name="thigh_max" value="3.5"/>
-    <xacro:property name="thigh_min" value="-1.0"/>
+    <xacro:property name="thigh_position_max" value="3.5"/>
+    <xacro:property name="thigh_position_min" value="-1.0"/>
     <xacro:property name="thigh_velocity_max" value="23.32"/>
     <xacro:property name="thigh_torque_max" value="93.33"/>
-    <xacro:property name="calf_max" value="-0.6"/>
-    <xacro:property name="calf_min" value="-2.6"/>
+    <xacro:property name="calf_position_max" value="-0.6"/>
+    <xacro:property name="calf_position_min" value="-2.6"/>
     <xacro:property name="calf_velocity_max" value="15.55"/>
     <xacro:property name="calf_torque_max" value="140"/>
@@ -66,4 +76,14 @@
     <xacro:property name="hip_iyz" value="0.00005638"/>
     <xacro:property name="hip_izz" value="0.00626340"/>
+    <xacro:property name="hip_rotor_mass" value="0.121"/><!-- 质心相对于hip转子的位置-->
+    <xacro:property name="hip_rotor_com_x" value="0.0"/>
+    <xacro:property name="hip_rotor_com_y" value="0.0"/>
+    <xacro:property name="hip_rotor_com_z" value="0.0"/>
+    <xacro:property name="hip_rotor_ixx" value="0.000103801"/>
+    <xacro:property name="hip_rotor_ixy" value="0.0"/>
+    <xacro:property name="hip_rotor_ixz" value="0.0"/>
+    <xacro:property name="hip_rotor_iyy" value="0.000054638"/>
+    <xacro:property name="hip_rotor_iyz" value="0.0"/>
+    <xacro:property name="hip_rotor_izz" value="0.000054638"/>
     <!-- thigh -->
     <xacro:property name="thigh_mass" value="2.459"/><!-- 重心相对于thigh关节的位置-->
@@ -77,4 +97,14 @@
     <xacro:property name="thigh_iyz" value="-0.00404389"/>
     <xacro:property name="thigh_izz" value="0.00849196"/>
+    <xacro:property name="thigh_rotor_mass" value="0.121"/>
+    <xacro:property name="thigh_rotor_com_x" value="0.0"/>
+    <xacro:property name="thigh_rotor_com_y" value="0.0"/>
+    <xacro:property name="thigh_rotor_com_z" value="0.0"/>
+    <xacro:property name="thigh_rotor_ixx" value="0.000103801"/>
+    <xacro:property name="thigh_rotor_ixy" value="0.0"/>
+    <xacro:property name="thigh_rotor_ixz" value="0.0"/>
+    <xacro:property name="thigh_rotor_iyy" value="0.000054638"/>
+    <xacro:property name="thigh_rotor_iyz" value="0.0"/>
+    <xacro:property name="thigh_rotor_izz" value="0.000054638"/>
     <!-- calf -->
     <xacro:property name="calf_mass" value="0.48137357"/><!-- 质心相对于calf关节的位置-->
@@ -88,4 +118,14 @@
     <xacro:property name="calf_iyz" value="0.00000137"/>
     <xacro:property name="calf_izz" value="0.00014153"/>
+    <xacro:property name="calf_rotor_mass" value="0.121"/>
+    <xacro:property name="calf_rotor_com_x" value="0.0"/>
+    <xacro:property name="calf_rotor_com_y" value="0.0"/>
+    <xacro:property name="calf_rotor_com_z" value="0.0"/>
+    <xacro:property name="calf_rotor_ixx" value="0.000103801"/>
+    <xacro:property name="calf_rotor_ixy" value="0.0"/>
+    <xacro:property name="calf_rotor_ixz" value="0.0"/>
+    <xacro:property name="calf_rotor_iyy" value="0.000054638"/>
+    <xacro:property name="calf_rotor_iyz" value="0.0"/>
+    <xacro:property name="calf_rotor_izz" value="0.000054638"/>
     <!-- foot -->
     <xacro:property name="foot_mass" value="0.05"/>

File: legged_examples/legged_unitree/legged_unitree_description/urdf/robot.xacro (robot description, xacro)
@@ -11,6 +11,20 @@
             <origin rpy="0 0 0" xyz="0 0 0"/>
             <geometry>
+                <box size="0.001 0.001 0.001"/>
+            </geometry>
+        </visual>
+    </link>
+    <joint name="floating_base" type="fixed">
+        <origin rpy="0 0 0" xyz="0 0 0"/>
+        <parent link="base"/>
+        <child link="trunk"/>
+    </joint>
+    <link name="trunk">
+        <visual>
+            <origin rpy="0 0 0" xyz="0 0 0"/>
+            <geometry>
                 <mesh filename="package://legged_unitree_description/meshes/$(arg robot_type)/trunk.dae" scale="1 1 1"/>
             </geometry>
+            <material name="orange"/>
         </visual>
         <collision>
@@ -30,15 +44,7 @@
     </link>
     <xacro:IMU connected_to="base" imu_name="unitree_imu" xyz="0. 0. 0." rpy="0. 0. 0."/>
-    <xacro:leg prefix="RF" mirror="-1" mirror_dae="False" front_hind="1" front_hind_dae="True">
-        <origin rpy="0 0 0" xyz="${leg_offset_x} ${-leg_offset_y} 0"/>
-    </xacro:leg>
-    <xacro:leg prefix="LF" mirror="1" mirror_dae="True" front_hind="1" front_hind_dae="True">
-        <origin rpy="0 0 0" xyz="${leg_offset_x} ${leg_offset_y} 0"/>
-    </xacro:leg>
-    <xacro:leg prefix="RH" mirror="-1" mirror_dae="False" front_hind="-1" front_hind_dae="False">
-        <origin rpy="0 0 0" xyz="${-leg_offset_x} ${-leg_offset_y} 0"/>
-    </xacro:leg>
-    <xacro:leg prefix="LH" mirror="1" mirror_dae="True" front_hind="-1" front_hind_dae="False">
-        <origin rpy="0 0 0" xyz="${-leg_offset_x} ${leg_offset_y} 0"/>
-    </xacro:leg>
+    <xacro:leg prefix="RF" mirror="-1" mirror_dae="False" front_hind="1" front_hind_dae="True"/>
+    <xacro:leg prefix="LF" mirror="1" mirror_dae="True" front_hind="1" front_hind_dae="True"/>
+    <xacro:leg prefix="RH" mirror="-1" mirror_dae="False" front_hind="-1" front_hind_dae="False"/>
+    <xacro:leg prefix="LH" mirror="1" mirror_dae="True" front_hind="-1" front_hind_dae="False"/>
 </robot>
